Commit message: Added launch file and gave gazebo properties to urdf file

File: description/robot_core.xacro (robot description, xacro)
@@ -41,4 +41,7 @@
 </xacro:inertial_box>
 </link>
+<gazebo references="chassis">
+<material>Gazebo/White</material>
+</gazebo>
 <joint name="left_wheel_joint" type="continuous">
 <parent link="base_link" />
@@ -63,4 +66,7 @@
 </xacro:inertial_box>
 </link>
+<gazebo references="left_wheel">
+<material>Gazebo/Blue</material>
+</gazebo>
 <joint name="right_wheel_joint" type="continuous">
 <parent link="base_link" />
@@ -85,4 +91,7 @@
 </xacro:inertial_box>
 </link>
+<gazebo references="right_wheel">
+<material>Gazebo/Blue</material>
+</gazebo>
 <joint name="caster_wheel_joint" type="fixed">
 <parent link="chassis" />
@@ -106,3 +115,6 @@
 </xacro:inertial_box>
 </link>
+<gazebo references="caster_wheel">
+<material>Gazebo/Black</material>
+</gazebo>
 </robot>
